File: PCH_Highspeed_Clock_LPC_eSPI.kicad_sch (KiCad schematic)
At the start: 1 part

Commit message: Titled PCH pages
Other:
- company: (none) -> WifiCable
- title: (none) -> PCH DMI, PCIe, SATA, USB3, USB2, Clockgen, CNVi, LPC/eSPI & GPIO
Changed lines of the file:
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@@
 	(generator_version "9.0")
 	(paper "A3")
+	(title_block
+		(title "PCH DMI, PCIe, SATA, USB3, USB2, Clockgen, CNVi, LPC/eSPI & GPIO")
+		(company "WifiCable")
+	)
 	(wire
 		(pts
