File: PCH_Lowspeed_SPI_HDA_GPIO.kicad_sch (KiCad schematic)
At the start: 1 part

Commit message: Titled PCH pages
Other:
- company: (none) -> WifiCable
- title: (none) -> PCH SPI, HDA/I2S, UART, I2C, SMBus, SML, HPD & GPIO
Changed lines of the file:
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@@
 	(generator_version "9.0")
 	(paper "A3")
+	(title_block
+		(title "PCH SPI, HDA/I2S, UART, I2C, SMBus, SML, HPD & GPIO")
+		(company "WifiCable")
+	)
 	(symbol
 		(lib_id "A-my-stuff:Intel_CFL_PCH_FCBGA874_but_better")
