File: PCH_Lowspeed_SPI_HDA_GPIO.kicad_sch (KiCad schematic)
At the start: 5 parts

Commit message: idek what i changed anymore but there's a bunch of new stuff lol
iirc i did some more misc cpu pins and a bunch of pch pcie stuff
Connections:
- net CPU_PWRGD: now reaches UPCH1.AE3 (CPUPWRGD)
Changed lines of the file:
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@@
 	(wire
 		(pts
+			(xy 261.62 115.57) (xy 256.54 115.57)
+		)
+		(stroke
+			(width 0)
+			(type default)
+		)
+	)
+	(wire
+		(pts
 			(xy 167.64 62.23) (xy 172.72 62.23)
 		)
@@
 		)
 	)
+	(global_label "CPU_PWRGD"
+		(shape output)
+		(at 261.62 115.57 0)
+		(fields_autoplaced yes)
+		(effects
+			(font
+				(size 1.27 1.27)
+			)
+			(justify left)
+		)
+		(property "Intersheetrefs" "${INTERSHEET_REFS}"
+			(at 275.9747 115.57 0)
+			(effects
+				(font
+					(size 1.27 1.27)
+				)
+				(justify left)
+				(hide yes)
+			)
+		)
+	)
 	(global_label "iGPU_DDI2_SCL"
 		(shape input)
@@
 		)
 		(instances
-			(project "Stroopwafel-LGA1151-CFL"
+			(project ""
+				(path "/4bc771b8-eb19-46d0-8798-27231a7c6e83/55a4f655-ea62-4675-bc34-60bbcfd07a2f"
+					(reference "UPCH1")
+					(unit 10)
+				)
 				(path "/4bc771b8-eb19-46d0-8798-27231a7c6e83/cd978078-9495-426d-921d-88f146c11707"
 					(reference "UPCH1")
@@
 		)
 		(instances
-			(project "Stroopwafel-LGA1151-CFL"
+			(project ""
+				(path "/4bc771b8-eb19-46d0-8798-27231a7c6e83/55a4f655-ea62-4675-bc34-60bbcfd07a2f"
+					(reference "UPCH1")
+					(unit 5)
+				)
 				(path "/4bc771b8-eb19-46d0-8798-27231a7c6e83/cd978078-9495-426d-921d-88f146c11707"
 					(reference "UPCH1")
@@
 		)
 		(instances
-			(project "Stroopwafel-LGA1151-CFL"
+			(project ""
+				(path "/4bc771b8-eb19-46d0-8798-27231a7c6e83/55a4f655-ea62-4675-bc34-60bbcfd07a2f"
+					(reference "UPCH1")
+					(unit 1)
+				)
 				(path "/4bc771b8-eb19-46d0-8798-27231a7c6e83/cd978078-9495-426d-921d-88f146c11707"
 					(reference "UPCH1")
@@
 		)
 		(instances
-			(project "Stroopwafel-LGA1151-CFL"
+			(project ""
+				(path "/4bc771b8-eb19-46d0-8798-27231a7c6e83/55a4f655-ea62-4675-bc34-60bbcfd07a2f"
+					(reference "UPCH1")
+					(unit 11)
+				)
 				(path "/4bc771b8-eb19-46d0-8798-27231a7c6e83/cd978078-9495-426d-921d-88f146c11707"
 					(reference "UPCH1")
@@
 		)
 		(instances
-			(project "Stroopwafel-LGA1151-CFL"
+			(project ""
+				(path "/4bc771b8-eb19-46d0-8798-27231a7c6e83/55a4f655-ea62-4675-bc34-60bbcfd07a2f"
+					(reference "UPCH1")
+					(unit 4)
+				)
 				(path "/4bc771b8-eb19-46d0-8798-27231a7c6e83/cd978078-9495-426d-921d-88f146c11707"
 					(reference "UPCH1")
