File: PCH_VCC_GND.kicad_sch (KiCad schematic)
At the start: 1 part

Commit message: Titled PCH pages
Other:
- company: (none) -> WifiCable
- title: (none) -> PCH VCC & GND
Changed lines of the file:
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@@
 	(generator_version "9.0")
 	(paper "A3")
+	(title_block
+		(title "PCH VCC & GND")
+		(company "WifiCable")
+	)
 	(junction
 		(at 361.95 54.61)
