File: Stroopwafel-LGA1151-CFL.kicad_pcb (KiCad board)
At the start: 2 copper layers, 49 parts, among them J1 PCIe_x16_CPU, J2 DP_A

Commit message: More DP
Parts:
- added C41: 0.1uF, Capacitor_SMD:C_0402_1005Metric, F.Cu at (243.5, 42.3)
- added C42: 0.1uF, Capacitor_SMD:C_0402_1005Metric, F.Cu at (245.5, 42.3)
- added C43: 0.1uF, Capacitor_SMD:C_0402_1005Metric, F.Cu at (247.4, 42.3)
- added C44: 0.1uF, Capacitor_SMD:C_0402_1005Metric, F.Cu at (249.4, 42.3)
- added C45: 0.1uF, Capacitor_SMD:C_0402_1005Metric, F.Cu at (243.5, 39.5)
- added C46: 0.1uF, Capacitor_SMD:C_0402_1005Metric, F.Cu at (245.5, 39.4)
- added C47: 0.1uF, Capacitor_SMD:C_0402_1005Metric, F.Cu at (247.4, 39.5)
- added C48: 0.1uF, Capacitor_SMD:C_0402_1005Metric, F.Cu at (249.4, 39.5)
- added C49: 0.1uF, Capacitor_SMD:C_0402_1005Metric, F.Cu at (223.9, 43.2)
- added C50: 0.1uF, Capacitor_SMD:C_0402_1005Metric, F.Cu at (225.9, 43.2)
- added C51: 0.1uF, Capacitor_SMD:C_0402_1005Metric, F.Cu at (227.9, 43.2)
- added C52: 0.1uF, Capacitor_SMD:C_0402_1005Metric, F.Cu at (229.9, 43.2)
- added C53: 0.1uF, Capacitor_SMD:C_0402_1005Metric, F.Cu at (223.9, 40.3)
- added C54: 0.1uF, Capacitor_SMD:C_0402_1005Metric, F.Cu at (225.9, 40.3)
- added C55: 0.1uF, Capacitor_SMD:C_0402_1005Metric, F.Cu at (227.9, 40.3)
- added C56: 0.1uF, Capacitor_SMD:C_0402_1005Metric, F.Cu at (229.9, 40.3)
- added J3: DP_B, A-my-stuff:DP-SMD_HYC16-DP20-178, F.Cu at (248.2, 30.7)
- added J4: DP_C, A-my-stuff:DP-SMD_HYC16-DP20-178, F.Cu at (227.2, 30.7)
- moved C33 35.7 mm to (262.1, 39.8)
- moved C35 35.7 mm to (266.0, 39.8)
- moved C37 35.7 mm to (270.0, 39.8)
- moved C39 35.7 mm to (273.9, 39.8)
- moved C34 35.7 mm to (264.1, 39.8)
- moved C36 35.7 mm to (268.0, 39.8)
- moved C38 35.7 mm to (272.0, 39.8)
- moved C40 35.7 mm to (275.9, 39.8)
- moved J2 35.7 mm to (269.2, 30.7)
Connections:
- JCPU1 pad A12: unconnected-(JCPU1D-DDI2_AUXP-PadA12) -> iGPU_DDI2_AUX+
- JCPU1 pad A14: unconnected-(JCPU1D-DDI3_TXN_0-PadA14) -> iGPU_DDI3_TX0-
- JCPU1 pad A16: unconnected-(JCPU1D-DDI3_TXN_2-PadA16) -> iGPU_DDI3_TX2-
- JCPU1 pad A18: unconnected-(JCPU1D-DDI2_TXN_0-PadA18) -> iGPU_DDI2_TX0-
- JCPU1 pad B11: unconnected-(JCPU1D-DDI3_AUXP-PadB11) -> iGPU_DDI3_AUX+
- JCPU1 pad B12: unconnected-(JCPU1D-DDI2_AUXN-PadB12) -> iGPU_DDI2_AUX-
- JCPU1 pad B14: unconnected-(JCPU1D-DDI3_TXP_0-PadB14) -> iGPU_DDI3_TX0+
- JCPU1 pad B15: unconnected-(JCPU1D-DDI3_TXN_1-PadB15) -> iGPU_DDI3_TX1-
- JCPU1 pad B16: unconnected-(JCPU1D-DDI3_TXP_2-PadB16) -> iGPU_DDI3_TX2+
- JCPU1 pad B17: unconnected-(JCPU1D-DDI3_TXN_3-PadB17) -> iGPU_DDI3_TX3-
- JCPU1 pad B18: unconnected-(JCPU1D-DDI2_TXP_0-PadB18) -> iGPU_DDI2_TX0+
- JCPU1 pad C11: unconnected-(JCPU1D-DDI3_AUXN-PadC11) -> iGPU_DDI3_AUX-
- JCPU1 pad C15: unconnected-(JCPU1D-DDI3_TXP_1-PadC15) -> iGPU_DDI3_TX1+
- JCPU1 pad C17: unconnected-(JCPU1D-DDI3_TXP_3-PadC17) -> iGPU_DDI3_TX3+
- JCPU1 pad C19: unconnected-(JCPU1D-DDI2_TXP_2-PadC19) -> iGPU_DDI2_TX2+
- JCPU1 pad D18: unconnected-(JCPU1D-DDI2_TXP_1-PadD18) -> iGPU_DDI2_TX1+
- JCPU1 pad D19: unconnected-(JCPU1D-DDI2_TXN_2-PadD19) -> iGPU_DDI2_TX2-
- JCPU1 pad D20: unconnected-(JCPU1D-DDI2_TXP_3-PadD20) -> iGPU_DDI2_TX3+
- JCPU1 pad E18: unconnected-(JCPU1D-DDI2_TXN_1-PadE18) -> iGPU_DDI2_TX1-
- JCPU1 pad E20: unconnected-(JCPU1D-DDI2_TXN_3-PadE20) -> iGPU_DDI2_TX3-
- UPCH1 pad AL10: unconnected-(UPCH1E-GPP_I8/DDPC_CTRLDATA-PadAL10) -> iGPU_DDI2_SDA
- UPCH1 pad AL9: unconnected-(UPCH1E-GPP_I9/DDPD_CTRLCLK-PadAL9) -> iGPU_DDI3_SCL
- UPCH1 pad AN13: unconnected-(UPCH1E-GPP_I7/DDPC_CTRLCLK-PadAN13) -> iGPU_DDI2_SCL
- UPCH1 pad AR3: unconnected-(UPCH1E-GPP_I10/DDPD_CTRLDATA-PadAR3) -> iGPU_DDI3_SDA

Commit message: partially added eDP + rearranged other display stuff
Parts:
- added C57: 0.1uF, Capacitor_SMD:C_0402_1005Metric, F.Cu at (274.7, 53.2)
- added C58: 0.1uF, Capacitor_SMD:C_0402_1005Metric, F.Cu at (275.4, 53.2)
- added Q1: 2N7002, Package_TO_SOT_SMD:SOT-23, F.Cu at (265.3, 48.5)
- added Q2: 2N7002, Package_TO_SOT_SMD:SOT-23, F.Cu at (264.4, 44.5)
- added Q3: 2N7002, Package_TO_SOT_SMD:SOT-23, F.Cu at (272.4, 48.1)
- added Q4: 2N7002, Package_TO_SOT_SMD:SOT-23, F.Cu at (275.8, 48.1)
- added Q5: 2N7002, Package_TO_SOT_SMD:SOT-23, F.Cu at (272.4, 44.1)
- added Q6: 2N7002, Package_TO_SOT_SMD:SOT-23, F.Cu at (275.8, 44.1)
- added R10: 24.9Ω_1%, Resistor_SMD:R_0402_1005Metric, F.Cu at (174.6, 56.4)
- added R11: 24.9Ω_1%, Resistor_SMD:R_0402_1005Metric, F.Cu at (174.5, 53.6)
- added R12: 49.9Ω_1%, Resistor_SMD:R_0402_1005Metric, F.Cu at (188.2, 47.0)
- added R4: 4.7kΩ?, Resistor_SMD:R_0402_1005Metric, F.Cu at (263.2, 49.9)
- added R5: 4.7kΩ?, Resistor_SMD:R_0402_1005Metric, F.Cu at (262.3, 45.9)
- added R6: 100kΩ, Resistor_SMD:R_0402_1005Metric, F.Cu at (271.2, 39.4)
- added R7: 100kΩ, Resistor_SMD:R_0402_1005Metric, F.Cu at (272.8, 39.4)
- added R8: 2.2kΩ, Resistor_SMD:R_0402_1005Metric, F.Cu at (268.2, 45.6)
- added R9: 2.2kΩ, Resistor_SMD:R_0402_1005Metric, F.Cu at (268.2, 46.6)
- moved C40 6.79 mm to (269.1, 39.3)
- moved C39 5.57 mm to (268.4, 39.3)
- moved C38 4.36 mm to (267.6, 39.3)
- moved C37 3.15 mm to (266.9, 39.3)
- moved C36 1.96 mm to (266.1, 39.3)
- moved C33 1.86 mm to (263.9, 39.3)
- moved C35 0.86 mm to (265.4, 39.3)
- moved C34 0.78 mm to (264.6, 39.3)
Connections:
- J2 pad 11: Net-(J2-GND-Pad11) -> GND
- J2 pad 13: unconnected-(J2-CONFIG1-Pad13) -> DP_A_Dongle_Det
- J2 pad 15: unconnected-(J2-AUX_CH_P-Pad15) -> DP_A_AUX+
- J2 pad 17: unconnected-(J2-AUX_CH_N-Pad17) -> DP_A_AUX-
- J2 pad 2: Net-(J2-GND-Pad11) -> GND
- J2 pad 21: Net-(J2-GND-Pad11) -> GND
- J2 pad 22: Net-(J2-GND-Pad11) -> GND
- J2 pad 23: Net-(J2-GND-Pad11) -> GND
- J2 pad 24: Net-(J2-GND-Pad11) -> GND
- J2 pad 5: Net-(J2-GND-Pad11) -> GND
- J2 pad 8: Net-(J2-GND-Pad11) -> GND
- J3 pad 11: Net-(J3-GND-Pad11) -> GND
- J3 pad 2: Net-(J3-GND-Pad11) -> GND
- J3 pad 21: Net-(J3-GND-Pad11) -> GND
- J3 pad 22: Net-(J3-GND-Pad11) -> GND
- J3 pad 23: Net-(J3-GND-Pad11) -> GND
- J3 pad 24: Net-(J3-GND-Pad11) -> GND
- J3 pad 5: Net-(J3-GND-Pad11) -> GND
- J3 pad 8: Net-(J3-GND-Pad11) -> GND
- J4 pad 11: Net-(J4-GND-Pad11) -> GND
- J4 pad 2: Net-(J4-GND-Pad11) -> GND
- J4 pad 21: Net-(J4-GND-Pad11) -> GND
- J4 pad 22: Net-(J4-GND-Pad11) -> GND
- J4 pad 23: Net-(J4-GND-Pad11) -> GND
- J4 pad 24: Net-(J4-GND-Pad11) -> GND
- J4 pad 5: Net-(J4-GND-Pad11) -> GND
- J4 pad 8: Net-(J4-GND-Pad11) -> GND
- JCPU1 pad L7: unconnected-(JCPU1C-PEG_RCOMP-PadL7) -> Net-(JCPU1C-PEG_RCOMP)
- JCPU1 pad M11: unconnected-(JCPU1E-CFG_RCOMP-PadM11) -> Net-(JCPU1E-CFG_RCOMP)
- JCPU1 pad M9: unconnected-(JCPU1D-DISP_RCOMP-PadM9) -> Net-(JCPU1D-DISP_RCOMP)
