File: Stroopwafel-LGA1151-CFL.kicad_pcb (KiCad board)
At the start: 2 copper layers, 118 parts, among them J1 PCIe_x16_CPU, J2 DP_A, J3 DP_B, J4 DP_C, J5 eDP 4-lane 40-pin ipex, Q1 2N7002, Q2 2N7002, Q3 2N7002, Q4 2N7002, Q5 2N7002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

Commit message: implemented some misc cpu signals
Parts:
- added D1: Really-bad-event-led, LED_SMD:LED_0603_1608Metric, F.Cu at (170.9, 49.6)
- added Q7: MMBT3904, Package_TO_SOT_SMD:SOT-23, F.Cu at (168.1, 47.7)
- added R35: 1kΩ, Resistor_SMD:R_0402_1005Metric, F.Cu at (165.5, 47.3)
- added R36: 1kΩ, Resistor_SMD:R_0402_1005Metric, F.Cu at (170.9, 46.9)
- added R37: 1kΩ, Resistor_SMD:R_0402_1005Metric, F.Cu at (106.4, 58.8)
- added R38: 619Ω, Resistor_SMD:R_0402_1005Metric, F.Cu at (104.5, 59.3)
- added R39: 0Ω, Resistor_SMD:R_0402_1005Metric, F.Cu at (101.5, 58.0)
- added R40: 43Ω, Resistor_SMD:R_0402_1005Metric, F.Cu at (81.9, 54.6)
- added R41: 1kΩ, Resistor_SMD:R_0402_1005Metric, F.Cu at (101.4, 59.5)
- added R42: 20Ω, Resistor_SMD:R_0402_1005Metric, F.Cu at (126.1, 59.6)
- added R43: 30Ω, Resistor_SMD:R_0402_1005Metric, F.Cu at (126.1, 61.6)
- added TP2: CFG-pullup-source-just-in-case, TestPoint:TestPoint_Pad_D2.0mm, F.Cu at (179.9, 40.0)
- added TP3: PROC_SELECT#, TestPoint:TestPoint_Pad_D2.0mm, F.Cu at (242.6, 75.0)
- moved R1 43.7 mm to (119.3, 57.3), turned to 180 degrees
- moved R2 43.7 mm to (119.3, 59.3), turned to 180 degrees
- moved R3 43.7 mm to (119.3, 61.3), turned to 180 degrees
- moved R33 41.8 mm to (98.4, 58.9)
- moved UPCH1 40.6 mm to (102.5, 75.2)
- moved R34 3.74 mm to (174.9, 52.6)
- moved R11 1.33 mm to (174.9, 54.9)
- moved R10 0.57 mm to (174.9, 55.9)
Connections:
- J1 pad A10: unconnected-(J1-+3.3V-PadA10) -> temp_3.3V
- J1 pad A2: unconnected-(J1-+12V-PadA2) -> temp_12V
- J1 pad A3: unconnected-(J1-+12V-PadA3) -> temp_12V
- J1 pad A9: unconnected-(J1-+3.3V-PadA9) -> temp_3.3V
- J1 pad B1: unconnected-(J1-+12V-PadB1) -> temp_12V
- J1 pad B2: unconnected-(J1-+12V-PadB2) -> temp_12V
- J1 pad B3: unconnected-(J1-+12V-PadB3) -> temp_12V
- J1 pad B8: unconnected-(J1-+3.3V-PadB8) -> temp_3.3V
- JCPU1 pad AB36: unconnected-(JCPU1E-PROC_SELECT#-PadAB36) -> Net-(JCPU1E-PROC_SELECT#)
- JCPU1 pad D11: unconnected-(JCPU1E-THERMTRIP#-PadD11) -> THERMTRIP#
- JCPU1 pad D13: unconnected-(JCPU1E-CATERR#-PadD13) -> CATERR#
- JCPU1 pad D8: unconnected-(JCPU1E-PM_DOWN-PadD8) -> Net-(JCPU1E-PM_DOWN)
- JCPU1 pad E7: unconnected-(JCPU1E-RESET#-PadE7) -> PLTRST_CPU#
- JCPU1 pad E8: unconnected-(JCPU1E-PM_SYNC-PadE8) -> Net-(JCPU1E-PM_SYNC)
- JCPU1 pad G7: unconnected-(JCPU1E-PECI-PadG7) -> Net-(JCPU1E-PECI)
- R11 pad 1: Net-(JCPU1D-DISP_RCOMP) -> VCCIO
- R11 pad 2: VCCIO -> Net-(JCPU1D-DISP_RCOMP)
- UPCH1 pad AD3: unconnected-(UPCH1C-THRMTRIP#-PadAD3) -> Net-(UPCH1C-THRMTRIP#)
- UPCH1 pad AE2: unconnected-(UPCH1C-PM_DOWN-PadAE2) -> PM_DOWN_PCH
- UPCH1 pad AF2: unconnected-(UPCH1C-PECI-PadAF2) -> PECI_PCH
- UPCH1 pad AF3: unconnected-(UPCH1C-PM_SYNC-PadAF3) -> PM_SYNC_PCH
- UPCH1 pad AG5: unconnected-(UPCH1C-PLTRST_CPU#-PadAG5) -> PLTRST_CPU#

Commit message: idek what i changed anymore but there's a bunch of new stuff lol
iirc i did some more misc cpu pins and a bunch of pch pcie stuff
Parts:
- added C69: 0.22uF, Capacitor_SMD:C_0402_1005Metric, F.Cu at (133.3, 96.5)
- added C70: 0.22uF, Capacitor_SMD:C_0402_1005Metric, F.Cu at (132.3, 96.5)
- added C71: 0.22uF, Capacitor_SMD:C_0402_1005Metric, F.Cu at (130.3, 96.5)
- added C72: 0.22uF, Capacitor_SMD:C_0402_1005Metric, F.Cu at (129.3, 96.5)
- added C73: 0.22uF, Capacitor_SMD:C_0402_1005Metric, F.Cu at (127.3, 96.5)
- added C74: 0.22uF, Capacitor_SMD:C_0402_1005Metric, F.Cu at (126.3, 96.5)
- added C75: 0.22uF, Capacitor_SMD:C_0402_1005Metric, F.Cu at (124.3, 96.5)
- added C76: 0.22uF, Capacitor_SMD:C_0402_1005Metric, F.Cu at (123.3, 96.5)
- added J6: Bus_M.2_Socket_M, A-my-stuff:m-key, F.Cu at (130.3, 104.5)
Connections:
- JCPU1 pad AC36: unconnected-(JCPU1E-DDR_VTT_CNTL-PadAC36) -> CPU_DDR_VTT_CNTL
- JCPU1 pad F8: unconnected-(JCPU1E-PROCPWRGD-PadF8) -> CPU_PWRGD
- JCPU1 pad U2: unconnected-(JCPU1E-VCCST_PWRGD-PadU2) -> CPU_VCCST_PWRGD
- UPCH1 pad AE3: unconnected-(UPCH1D-CPUPWRGD-PadAE3) -> CPU_PWRGD
- UPCH1 pad AH10: unconnected-(UPCH1G-CLKOUT_PCIE_P1-PadAH10) -> SSD0_Refclk+
- UPCH1 pad AH9: unconnected-(UPCH1G-CLKOUT_PCIE_N1-PadAH9) -> SSD0_Refclk-
- UPCH1 pad B35: unconnected-(UPCH1C-PCIE10_TXP-PadB35) -> SSD0_PCIe_Tx2+
- UPCH1 pad B36: unconnected-(UPCH1C-PCIE11_TXN/SATA0A_TXN-PadB36) -> SSD0_PCIe_Tx1-
- UPCH1 pad BE31: unconnected-(UPCH1G-GPP_B6/SRCCLKREQ1#-PadBE31) -> SSD0_CLKREQ#
- UPCH1 pad C34: unconnected-(UPCH1C-PCIE9_TXN-PadC34) -> SSD0_PCIe_Tx3-
- UPCH1 pad C35: unconnected-(UPCH1C-PCIE10_TXN-PadC35) -> SSD0_PCIe_Tx2-
- UPCH1 pad C36: unconnected-(UPCH1C-PCIE11_TXP/SATA0A_TXP-PadC36) -> SSD0_PCIe_Tx1+
- UPCH1 pad D34: unconnected-(UPCH1C-PCIE9_TXP-PadD34) -> SSD0_PCIe_Tx3+
- UPCH1 pad D38: unconnected-(UPCH1C-PCIE12_TXN/SATA1A_TXN-PadD38) -> SSD0_PCIe/SATA_Tx0-
- UPCH1 pad E37: unconnected-(UPCH1C-PCIE12_TXP/SATA1A_TXP-PadE37) -> SSD0_PCIe/SATA_Tx0+
- UPCH1 pad F36: unconnected-(UPCH1C-PCIE9_RXP-PadF36) -> SSD0_PCIe_Rx3+
- UPCH1 pad F39: unconnected-(UPCH1C-PCIE11_RXP/SATA0A_RXP-PadF39) -> SSD0_PCIe_Rx1+
- UPCH1 pad G36: unconnected-(UPCH1C-PCIE9_RXN-PadG36) -> SSD0_PCIe_Rx3-
- UPCH1 pad G38: unconnected-(UPCH1C-PCIE11_RXN/SATA0A_RXN-PadG38) -> SSD0_PCIe_Rx1-
- UPCH1 pad H42: unconnected-(UPCH1C-PCIE12_RXN/SATA1A_RXN-PadH42) -> SSD0_PCIe/SATA_Rx0-
- UPCH1 pad J37: unconnected-(UPCH1C-PCIE10_RXP-PadJ37) -> SSD0_PCIe_Rx2+
- UPCH1 pad J41: unconnected-(UPCH1C-PCIE12_RXP/SATA1A_RXP-PadJ41) -> SSD0_PCIe/SATA_Rx0+
- UPCH1 pad K37: unconnected-(UPCH1C-PCIE10_RXN-PadK37) -> SSD0_PCIe_Rx2-
