File: CPU_Display.kicad_sch (KiCad schematic)
At the start: 2 parts

Commit message: Added LGA1151 socket bracket holes
stolen from another lga1151 footprint that has wrong pin numbers....
Parts:
- JCPU1: footprint A-my-stuff:LGA-1151_L47.1-W42.5-P0.91_PE115127-4041-01H -> A-my-stuff:LGA1151_TE-2287402-1
Changed lines of the file:
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@@
 			)
 		)
-		(property "Footprint" "A-my-stuff:LGA-1151_L47.1-W42.5-P0.91_PE115127-4041-01H"
+		(property "Footprint" "A-my-stuff:LGA1151_TE-2287402-1"
 			(at 148.59 250.19 0)
 			(effects

Commit message: Added CPU CFG resistors
Parts:
- JCPU1: footprint A-my-stuff:LGA1151_TE-2287402-1 -> A-my-stuff:LGA-1151_L47.1-W42.5-P0.91_PE115127-4041-01H
Changed lines of the file:
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@@
 			)
 		)
-		(property "Footprint" "A-my-stuff:LGA1151_TE-2287402-1"
+		(property "Footprint" "A-my-stuff:LGA-1151_L47.1-W42.5-P0.91_PE115127-4041-01H"
 			(at 148.59 250.19 0)
 			(effects
