File: DDR4_slots.kicad_sch (KiCad schematic)
At the start: 0 parts

Commit message: Added DP_A DP++ HDMI dongle detection circuit
Parts:
- added JSODIMM1, JSODIMM2: DDR4-sodimm, A-my-stuff:DDR4-sodimm-std, symbol A-my-stuff:DDR4-sodimm
Connections:
- new net DDR4_CH0_A0: JSODIMM1.144 (A0)
- new net DDR4_CH0_A1: JSODIMM1.133 (A1)
- new net DDR4_CH0_A10: JSODIMM1.146 (A10/AP)
- new net DDR4_CH0_A11: JSODIMM1.120 (A11)
- new net DDR4_CH0_A12: JSODIMM1.119 (A12/BC#)
- new net DDR4_CH0_A13: JSODIMM1.158 (A13)
- new net DDR4_CH0_A14_WE#: JSODIMM1.151 (A14/WE#)
- new net DDR4_CH0_A15_CAS#: JSODIMM1.156 (A15/CAS#)
- new net DDR4_CH0_A16_RAS#: JSODIMM1.152 (A16/RAS#)
- new net DDR4_CH0_A2: JSODIMM1.132 (A2)
- new net DDR4_CH0_A3: JSODIMM1.131 (A3)
- new net DDR4_CH0_A4: JSODIMM1.128 (A4)
- new net DDR4_CH0_A5: JSODIMM1.126 (A5)
- new net DDR4_CH0_A6: JSODIMM1.127 (A6)
- new net DDR4_CH0_A7: JSODIMM1.122 (A7)
- new net DDR4_CH0_A8: JSODIMM1.125 (A8)
- new net DDR4_CH0_A9: JSODIMM1.121 (A9)
- new net DDR4_CH0_ACT#: JSODIMM1.114 (ACT#)
- new net DDR4_CH0_Alert#: JSODIMM1.116 (ALERT#)
- new net DDR4_CH0_BA0: JSODIMM1.150 (BA0)
- new net DDR4_CH0_BA1: JSODIMM1.145 (BA1)
- new net DDR4_CH0_BG0: JSODIMM1.115 (BG0)
- new net DDR4_CH0_BG1: JSODIMM1.113 (BG1)
- new net DDR4_CH0_CKE0: JSODIMM1.109 (CKE0)
- new net DDR4_CH0_CKE1: JSODIMM1.110 (CKE1)
- new net DDR4_CH0_CLK0+: JSODIMM1.137 (CK0+)
- new net DDR4_CH0_CLK0-: JSODIMM1.139 (CK0-)
- new net DDR4_CH0_CLK1+: JSODIMM1.138 (CK1+)
- new net DDR4_CH0_CLK1-: JSODIMM1.140 (CK1-)
- new net DDR4_CH0_CS0#: JSODIMM1.149 (CS0#)
- new net DDR4_CH0_CS1#: JSODIMM1.157 (CS1#)
- new net DDR4_CH0_DQ0: JSODIMM1.8 (DQ0)
- new net DDR4_CH0_DQ1: JSODIMM1.7 (DQ1)
- new net DDR4_CH0_DQ10: JSODIMM1.41 (DQ10)
- new net DDR4_CH0_DQ11: JSODIMM1.42 (DQ11)
- new net DDR4_CH0_DQ12: JSODIMM1.24 (DQ12)
- new net DDR4_CH0_DQ13: JSODIMM1.25 (DQ13)
- new net DDR4_CH0_DQ14: JSODIMM1.38 (DQ14)
- new net DDR4_CH0_DQ15: JSODIMM1.37 (DQ15)
- new net DDR4_CH0_DQ16: JSODIMM1.50 (DQ16)
- new net DDR4_CH0_DQ17: JSODIMM1.49 (DQ17)
- new net DDR4_CH0_DQ18: JSODIMM1.62 (DQ18)
- new net DDR4_CH0_DQ19: JSODIMM1.63 (DQ19)
- new net DDR4_CH0_DQ2: JSODIMM1.20 (DQ2)
- new net DDR4_CH0_DQ20: JSODIMM1.46 (DQ20)
- new net DDR4_CH0_DQ21: JSODIMM1.45 (DQ21)
- new net DDR4_CH0_DQ22: JSODIMM1.58 (DQ22)
- new net DDR4_CH0_DQ23: JSODIMM1.59 (DQ23)
- new net DDR4_CH0_DQ24: JSODIMM1.70 (DQ24)
- new net DDR4_CH0_DQ25: JSODIMM1.71 (DQ25)
- new net DDR4_CH0_DQ26: JSODIMM1.83 (DQ26)
- new net DDR4_CH0_DQ27: JSODIMM1.84 (DQ27)
- new net DDR4_CH0_DQ28: JSODIMM1.66 (DQ28)
- new net DDR4_CH0_DQ29: JSODIMM1.67 (DQ29)
- new net DDR4_CH0_DQ3: JSODIMM1.21 (DQ3)
- new net DDR4_CH0_DQ30: JSODIMM1.79 (DQ30)
- new net DDR4_CH0_DQ31: JSODIMM1.80 (DQ31)
- new net DDR4_CH0_DQ32: JSODIMM1.174 (DQ32)
- new net DDR4_CH0_DQ33: JSODIMM1.173 (DQ33)
- new net DDR4_CH0_DQ34: JSODIMM1.187 (DQ34)
- new net DDR4_CH0_DQ35: JSODIMM1.186 (DQ35)
- new net DDR4_CH0_DQ36: JSODIMM1.170 (DQ36)
- new net DDR4_CH0_DQ37: JSODIMM1.169 (DQ37)
- new net DDR4_CH0_DQ38: JSODIMM1.183 (DQ38)
- new net DDR4_CH0_DQ39: JSODIMM1.182 (DQ39)
- new net DDR4_CH0_DQ4: JSODIMM1.4 (DQ4)
- new net DDR4_CH0_DQ40: JSODIMM1.195 (DQ40)
- new net DDR4_CH0_DQ41: JSODIMM1.194 (DQ41)
- new net DDR4_CH0_DQ42: JSODIMM1.207 (DQ42)
- new net DDR4_CH0_DQ43: JSODIMM1.208 (DQ43)
- new net DDR4_CH0_DQ44: JSODIMM1.191 (DQ44)
- new net DDR4_CH0_DQ45: JSODIMM1.190 (DQ45)
- new net DDR4_CH0_DQ46: JSODIMM1.203 (DQ46)
- new net DDR4_CH0_DQ47: JSODIMM1.204 (DQ47)
- new net DDR4_CH0_DQ48: JSODIMM1.216 (DQ48)
- new net DDR4_CH0_DQ49: JSODIMM1.215 (DQ49)
- new net DDR4_CH0_DQ5: JSODIMM1.3 (DQ5)
- new net DDR4_CH0_DQ50: JSODIMM1.228 (DQ50)
- new net DDR4_CH0_DQ51: JSODIMM1.229 (DQ51)
- new net DDR4_CH0_DQ52: JSODIMM1.211 (DQ52)
- new net DDR4_CH0_DQ53: JSODIMM1.212 (DQ53)
- new net DDR4_CH0_DQ54: JSODIMM1.224 (DQ54)
- new net DDR4_CH0_DQ55: JSODIMM1.225 (DQ55)
- new net DDR4_CH0_DQ56: JSODIMM1.237 (DQ56)
- new net DDR4_CH0_DQ57: JSODIMM1.236 (DQ57)
- new net DDR4_CH0_DQ58: JSODIMM1.249 (DQ58)
- new net DDR4_CH0_DQ59: JSODIMM1.250 (DQ59)
- new net DDR4_CH0_DQ6: JSODIMM1.16 (DQ6)
- new net DDR4_CH0_DQ60: JSODIMM1.232 (DQ60)
- new net DDR4_CH0_DQ61: JSODIMM1.233 (DQ61)
- new net DDR4_CH0_DQ62: JSODIMM1.245 (DQ62)
- new net DDR4_CH0_DQ63: JSODIMM1.246 (DQ63)
- new net DDR4_CH0_DQ7: JSODIMM1.17 (DQ7)
- new net DDR4_CH0_DQ8: JSODIMM1.28 (DQ8)
- new net DDR4_CH0_DQ9: JSODIMM1.29 (DQ9)
- new net DDR4_CH0_DQS0+: JSODIMM1.13 (DQS0+)
- new net DDR4_CH0_DQS0-: JSODIMM1.11 (DQS0-)
- new net DDR4_CH0_DQS1+: JSODIMM1.34 (DQS1+)
- new net DDR4_CH0_DQS1-: JSODIMM1.32 (DQS1-)
- new net DDR4_CH0_DQS2+: JSODIMM1.55 (DQS2+)
- new net DDR4_CH0_DQS2-: JSODIMM1.53 (DQS2-)
- new net DDR4_CH0_DQS3+: JSODIMM1.76 (DQS3+)
- new net DDR4_CH0_DQS3-: JSODIMM1.74 (DQS3-)
- new net DDR4_CH0_DQS4+: JSODIMM1.179 (DQS4+)
- new net DDR4_CH0_DQS4-: JSODIMM1.177 (DQS4-)
- new net DDR4_CH0_DQS5+: JSODIMM1.200 (DQS5+)
- new net DDR4_CH0_DQS5-: JSODIMM1.198 (DQS5-)
- new net DDR4_CH0_DQS6+: JSODIMM1.221 (DQS6+)
- new net DDR4_CH0_DQS6-: JSODIMM1.219 (DQS6-)
- new net DDR4_CH0_DQS7+: JSODIMM1.242 (DQS7+)
- new net DDR4_CH0_DQS7-: JSODIMM1.240 (DQS7-)
- new net DDR4_CH0_DQS8+: JSODIMM1.97 (DQS8+)
- new net DDR4_CH0_DQS8-: JSODIMM1.95 (DQS8-)
- new net DDR4_CH0_ECC0: JSODIMM1.92 (CB0)
- new net DDR4_CH0_ECC1: JSODIMM1.91 (CB1)
- new net DDR4_CH0_ECC2: JSODIMM1.101 (CB2)
- new net DDR4_CH0_ECC3: JSODIMM1.105 (CB3)
- new net DDR4_CH0_ECC4: JSODIMM1.88 (CB4)
- new net DDR4_CH0_ECC5: JSODIMM1.87 (CB5)
- new net DDR4_CH0_ECC6: JSODIMM1.100 (CB6)
- new net DDR4_CH0_ECC7: JSODIMM1.104 (CB7)
- new net DDR4_CH0_ODT0: JSODIMM1.155 (ODT0)
- new net DDR4_CH0_ODT1: JSODIMM1.161 (ODT1)
- new net DDR4_CH0_Parity: JSODIMM1.143 (PARITY)
- new net DDR4_CH1_A0: JSODIMM2.144 (A0)
- new net DDR4_CH1_A1: JSODIMM2.133 (A1)
- new net DDR4_CH1_A10: JSODIMM2.146 (A10/AP)
- new net DDR4_CH1_A11: JSODIMM2.120 (A11)
- new net DDR4_CH1_A12: JSODIMM2.119 (A12/BC#)
- new net DDR4_CH1_A13: JSODIMM2.158 (A13)
- new net DDR4_CH1_A14_WE#: JSODIMM2.151 (A14/WE#)
- new net DDR4_CH1_A15_CAS#: JSODIMM2.156 (A15/CAS#)
- new net DDR4_CH1_A16_RAS#: JSODIMM2.152 (A16/RAS#)
- new net DDR4_CH1_A2: JSODIMM2.132 (A2)
- new net DDR4_CH1_A3: JSODIMM2.131 (A3)
- new net DDR4_CH1_A4: JSODIMM2.128 (A4)
- new net DDR4_CH1_A5: JSODIMM2.126 (A5)
- new net DDR4_CH1_A6: JSODIMM2.127 (A6)
- new net DDR4_CH1_A7: JSODIMM2.122 (A7)
- new net DDR4_CH1_A8: JSODIMM2.125 (A8)
- new net DDR4_CH1_A9: JSODIMM2.121 (A9)
- new net DDR4_CH1_ACT#: JSODIMM2.114 (ACT#)
- new net DDR4_CH1_Alert#: JSODIMM2.116 (ALERT#)
- new net DDR4_CH1_BA0: JSODIMM2.150 (BA0)
- new net DDR4_CH1_BA1: JSODIMM2.145 (BA1)
- new net DDR4_CH1_BG0: JSODIMM2.115 (BG0)
- new net DDR4_CH1_BG1: JSODIMM2.113 (BG1)
- new net DDR4_CH1_CKE0: JSODIMM2.109 (CKE0)
- new net DDR4_CH1_CKE1: JSODIMM2.110 (CKE1)
- new net DDR4_CH1_CLK0+: JSODIMM2.137 (CK0+)
- new net DDR4_CH1_CLK0-: JSODIMM2.139 (CK0-)
- new net DDR4_CH1_CLK1+: JSODIMM2.138 (CK1+)
- new net DDR4_CH1_CLK1-: JSODIMM2.140 (CK1-)
- new net DDR4_CH1_CS0#: JSODIMM2.149 (CS0#)
- new net DDR4_CH1_CS1#: JSODIMM2.157 (CS1#)
- new net DDR4_CH1_DQ0: JSODIMM2.8 (DQ0)
- new net DDR4_CH1_DQ1: JSODIMM2.7 (DQ1)
- new net DDR4_CH1_DQ10: JSODIMM2.41 (DQ10)
- new net DDR4_CH1_DQ11: JSODIMM2.42 (DQ11)
- new net DDR4_CH1_DQ12: JSODIMM2.24 (DQ12)
- new net DDR4_CH1_DQ13: JSODIMM2.25 (DQ13)
- new net DDR4_CH1_DQ14: JSODIMM2.38 (DQ14)
- new net DDR4_CH1_DQ15: JSODIMM2.37 (DQ15)
- new net DDR4_CH1_DQ16: JSODIMM2.50 (DQ16)
- new net DDR4_CH1_DQ17: JSODIMM2.49 (DQ17)
- new net DDR4_CH1_DQ18: JSODIMM2.62 (DQ18)
- new net DDR4_CH1_DQ19: JSODIMM2.63 (DQ19)
- new net DDR4_CH1_DQ2: JSODIMM2.20 (DQ2)
- new net DDR4_CH1_DQ20: JSODIMM2.46 (DQ20)
- new net DDR4_CH1_DQ21: JSODIMM2.45 (DQ21)
- new net DDR4_CH1_DQ22: JSODIMM2.58 (DQ22)
- new net DDR4_CH1_DQ23: JSODIMM2.59 (DQ23)
- new net DDR4_CH1_DQ24: JSODIMM2.70 (DQ24)
- new net DDR4_CH1_DQ25: JSODIMM2.71 (DQ25)
- new net DDR4_CH1_DQ26: JSODIMM2.83 (DQ26)
- new net DDR4_CH1_DQ27: JSODIMM2.84 (DQ27)
- new net DDR4_CH1_DQ28: JSODIMM2.66 (DQ28)
- new net DDR4_CH1_DQ29: JSODIMM2.67 (DQ29)
- new net DDR4_CH1_DQ3: JSODIMM2.21 (DQ3)
- new net DDR4_CH1_DQ30: JSODIMM2.79 (DQ30)
- new net DDR4_CH1_DQ31: JSODIMM2.80 (DQ31)
- new net DDR4_CH1_DQ32: JSODIMM2.174 (DQ32)
- new net DDR4_CH1_DQ33: JSODIMM2.173 (DQ33)
- new net DDR4_CH1_DQ34: JSODIMM2.187 (DQ34)
- new net DDR4_CH1_DQ35: JSODIMM2.186 (DQ35)
- new net DDR4_CH1_DQ36: JSODIMM2.170 (DQ36)
- new net DDR4_CH1_DQ37: JSODIMM2.169 (DQ37)
- new net DDR4_CH1_DQ38: JSODIMM2.183 (DQ38)
- new net DDR4_CH1_DQ39: JSODIMM2.182 (DQ39)
- new net DDR4_CH1_DQ4: JSODIMM2.4 (DQ4)
- new net DDR4_CH1_DQ40: JSODIMM2.195 (DQ40)
- new net DDR4_CH1_DQ41: JSODIMM2.194 (DQ41)
- new net DDR4_CH1_DQ42: JSODIMM2.207 (DQ42)
- new net DDR4_CH1_DQ43: JSODIMM2.208 (DQ43)
- new net DDR4_CH1_DQ44: JSODIMM2.191 (DQ44)
- new net DDR4_CH1_DQ45: JSODIMM2.190 (DQ45)
- new net DDR4_CH1_DQ46: JSODIMM2.203 (DQ46)
- new net DDR4_CH1_DQ47: JSODIMM2.204 (DQ47)
- new net DDR4_CH1_DQ48: JSODIMM2.216 (DQ48)
- new net DDR4_CH1_DQ49: JSODIMM2.215 (DQ49)
- new net DDR4_CH1_DQ5: JSODIMM2.3 (DQ5)
- new net DDR4_CH1_DQ50: JSODIMM2.228 (DQ50)
- new net DDR4_CH1_DQ51: JSODIMM2.229 (DQ51)
- new net DDR4_CH1_DQ52: JSODIMM2.211 (DQ52)
- new net DDR4_CH1_DQ53: JSODIMM2.212 (DQ53)
- new net DDR4_CH1_DQ54: JSODIMM2.224 (DQ54)
- new net DDR4_CH1_DQ55: JSODIMM2.225 (DQ55)
- new net DDR4_CH1_DQ56: JSODIMM2.237 (DQ56)
- new net DDR4_CH1_DQ57: JSODIMM2.236 (DQ57)
- new net DDR4_CH1_DQ58: JSODIMM2.249 (DQ58)
- new net DDR4_CH1_DQ59: JSODIMM2.250 (DQ59)
- new net DDR4_CH1_DQ6: JSODIMM2.16 (DQ6)
- new net DDR4_CH1_DQ60: JSODIMM2.232 (DQ60)
- new net DDR4_CH1_DQ61: JSODIMM2.233 (DQ61)
- new net DDR4_CH1_DQ62: JSODIMM2.245 (DQ62)
- new net DDR4_CH1_DQ63: JSODIMM2.246 (DQ63)
- new net DDR4_CH1_DQ7: JSODIMM2.17 (DQ7)
- new net DDR4_CH1_DQ8: JSODIMM2.28 (DQ8)
- new net DDR4_CH1_DQ9: JSODIMM2.29 (DQ9)
- new net DDR4_CH1_DQS0+: JSODIMM2.13 (DQS0+)
- new net DDR4_CH1_DQS0-: JSODIMM2.11 (DQS0-)
- new net DDR4_CH1_DQS1+: JSODIMM2.34 (DQS1+)
- new net DDR4_CH1_DQS1-: JSODIMM2.32 (DQS1-)
- new net DDR4_CH1_DQS2+: JSODIMM2.55 (DQS2+)
- new net DDR4_CH1_DQS2-: JSODIMM2.53 (DQS2-)
- new net DDR4_CH1_DQS3+: JSODIMM2.76 (DQS3+)
- new net DDR4_CH1_DQS3-: JSODIMM2.74 (DQS3-)
- new net DDR4_CH1_DQS4+: JSODIMM2.179 (DQS4+)
- new net DDR4_CH1_DQS4-: JSODIMM2.177 (DQS4-)
- new net DDR4_CH1_DQS5+: JSODIMM2.200 (DQS5+)
- new net DDR4_CH1_DQS5-: JSODIMM2.198 (DQS5-)
- new net DDR4_CH1_DQS6+: JSODIMM2.221 (DQS6+)
- new net DDR4_CH1_DQS6-: JSODIMM2.219 (DQS6-)
- new net DDR4_CH1_DQS7+: JSODIMM2.242 (DQS7+)
- new net DDR4_CH1_DQS7-: JSODIMM2.240 (DQS7-)
- new net DDR4_CH1_DQS8+: JSODIMM2.97 (DQS8+)
- new net DDR4_CH1_DQS8-: JSODIMM2.95 (DQS8-)
- new net DDR4_CH1_ECC0: JSODIMM2.92 (CB0)
- new net DDR4_CH1_ECC1: JSODIMM2.91 (CB1)
- new net DDR4_CH1_ECC2: JSODIMM2.101 (CB2)
- new net DDR4_CH1_ECC3: JSODIMM2.105 (CB3)
- new net DDR4_CH1_ECC4: JSODIMM2.88 (CB4)
- new net DDR4_CH1_ECC5: JSODIMM2.87 (CB5)
- new net DDR4_CH1_ECC6: JSODIMM2.100 (CB6)
- new net DDR4_CH1_ECC7: JSODIMM2.104 (CB7)
- new net DDR4_CH1_ODT0: JSODIMM2.155 (ODT0)
- new net DDR4_CH1_ODT1: JSODIMM2.161 (ODT1)
- new net DDR4_CH1_Parity: JSODIMM2.143 (PARITY)
- new net GND: JSODIMM1.1 (VSS), JSODIMM1.10 (VSS), JSODIMM1.102 (VSS), JSODIMM1.103 (VSS), JSODIMM1.106 (VSS), JSODIMM1.107 (VSS), JSODIMM1.14 (VSS), JSODIMM1.15 (VSS), JSODIMM1.167 (VSS), JSODIMM1.168 (VSS), JSODIMM1.171 (VSS), JSODIMM1.172 (VSS), JSODIMM1.175 (VSS), JSODIMM1.176 (VSS), JSODIMM1.18 (VSS), JSODIMM1.180 (VSS), JSODIMM1.181 (VSS), JSODIMM1.184 (VSS), JSODIMM1.185 (VSS), JSODIMM1.188 (VSS), JSODIMM1.189 (VSS), JSODIMM1.19 (VSS), JSODIMM1.192 (VSS), JSODIMM1.193 (VSS), JSODIMM1.196 (VSS), JSODIMM1.197 (VSS), JSODIMM1.2 (VSS), JSODIMM1.201 (VSS), JSODIMM1.202 (VSS), JSODIMM1.205 (VSS), JSODIMM1.206 (VSS), JSODIMM1.209 (VSS), JSODIMM1.210 (VSS), JSODIMM1.213 (VSS), JSODIMM1.214 (VSS), JSODIMM1.217 (VSS), JSODIMM1.218 (VSS), JSODIMM1.22 (VSS), JSODIMM1.222 (VSS), JSODIMM1.223 (VSS), JSODIMM1.226 (VSS), JSODIMM1.227 (VSS), JSODIMM1.23 (VSS), JSODIMM1.230 (VSS), JSODIMM1.231 (VSS), JSODIMM1.234 (VSS), JSODIMM1.235 (VSS), JSODIMM1.238 (VSS), JSODIMM1.239 (VSS), JSODIMM1.243 (VSS), JSODIMM1.244 (VSS), JSODIMM1.247 (VSS), JSODIMM1.248 (VSS), JSODIMM1.251 (VSS), JSODIMM1.252 (VSS), JSODIMM1.26 (VSS), JSODIMM1.27 (VSS), JSODIMM1.30 (VSS), JSODIMM1.31 (VSS), JSODIMM1.35 (VSS), JSODIMM1.36 (VSS), JSODIMM1.39 (VSS), JSODIMM1.40 (VSS), JSODIMM1.43 (VSS), JSODIMM1.44 (VSS), JSODIMM1.47 (VSS), JSODIMM1.48 (VSS), JSODIMM1.5 (VSS), JSODIMM1.51 (VSS), JSODIMM1.52 (VSS), JSODIMM1.56 (VSS), JSODIMM1.57 (VSS), JSODIMM1.6 (VSS), JSODIMM1.60 (VSS), JSODIMM1.61 (VSS), JSODIMM1.64 (VSS), JSODIMM1.65 (VSS), JSODIMM1.68 (VSS), JSODIMM1.69 (VSS), JSODIMM1.72 (VSS), JSODIMM1.73 (VSS), JSODIMM1.77 (VSS), JSODIMM1.78 (VSS), JSODIMM1.81 (VSS), JSODIMM1.82 (VSS), JSODIMM1.85 (VSS), JSODIMM1.86 (VSS), JSODIMM1.89 (VSS), JSODIMM1.9 (VSS), JSODIMM1.90 (VSS), JSODIMM1.93 (VSS), JSODIMM1.94 (VSS), JSODIMM1.98 (VSS), JSODIMM1.99 (VSS), JSODIMM1.MP1, JSODIMM1.MP2, JSODIMM2.1 (VSS), JSODIMM2.10 (VSS), JSODIMM2.102 (VSS), JSODIMM2.103 (VSS), JSODIMM2.106 (VSS), JSODIMM2.107 (VSS), JSODIMM2.14 (VSS), JSODIMM2.15 (VSS), JSODIMM2.167 (VSS), JSODIMM2.168 (VSS), JSODIMM2.171 (VSS), JSODIMM2.172 (VSS), JSODIMM2.175 (VSS), JSODIMM2.176 (VSS), JSODIMM2.18 (VSS), JSODIMM2.180 (VSS), JSODIMM2.181 (VSS), JSODIMM2.184 (VSS), JSODIMM2.185 (VSS), JSODIMM2.188 (VSS), JSODIMM2.189 (VSS), JSODIMM2.19 (VSS), JSODIMM2.192 (VSS), JSODIMM2.193 (VSS), JSODIMM2.196 (VSS), JSODIMM2.197 (VSS), JSODIMM2.2 (VSS), JSODIMM2.201 (VSS), JSODIMM2.202 (VSS), JSODIMM2.205 (VSS), JSODIMM2.206 (VSS), JSODIMM2.209 (VSS), JSODIMM2.210 (VSS), JSODIMM2.213 (VSS), JSODIMM2.214 (VSS), JSODIMM2.217 (VSS), JSODIMM2.218 (VSS), JSODIMM2.22 (VSS), JSODIMM2.222 (VSS), JSODIMM2.223 (VSS), JSODIMM2.226 (VSS), JSODIMM2.227 (VSS), JSODIMM2.23 (VSS), JSODIMM2.230 (VSS), JSODIMM2.231 (VSS), JSODIMM2.234 (VSS), JSODIMM2.235 (VSS), JSODIMM2.238 (VSS), JSODIMM2.239 (VSS), JSODIMM2.243 (VSS), JSODIMM2.244 (VSS), JSODIMM2.247 (VSS), JSODIMM2.248 (VSS), JSODIMM2.251 (VSS), JSODIMM2.252 (VSS), JSODIMM2.26 (VSS), JSODIMM2.27 (VSS), JSODIMM2.30 (VSS), JSODIMM2.31 (VSS), JSODIMM2.35 (VSS), JSODIMM2.36 (VSS), JSODIMM2.39 (VSS), JSODIMM2.40 (VSS), JSODIMM2.43 (VSS), JSODIMM2.44 (VSS), JSODIMM2.47 (VSS), JSODIMM2.48 (VSS), JSODIMM2.5 (VSS), JSODIMM2.51 (VSS), JSODIMM2.52 (VSS), JSODIMM2.56 (VSS), JSODIMM2.57 (VSS), JSODIMM2.6 (VSS), JSODIMM2.60 (VSS), JSODIMM2.61 (VSS), JSODIMM2.64 (VSS), JSODIMM2.65 (VSS), JSODIMM2.68 (VSS), JSODIMM2.69 (VSS), JSODIMM2.72 (VSS), JSODIMM2.73 (VSS), JSODIMM2.77 (VSS), JSODIMM2.78 (VSS), JSODIMM2.81 (VSS), JSODIMM2.82 (VSS), JSODIMM2.85 (VSS), JSODIMM2.86 (VSS), JSODIMM2.89 (VSS), JSODIMM2.9 (VSS), JSODIMM2.90 (VSS), JSODIMM2.93 (VSS), JSODIMM2.94 (VSS), JSODIMM2.98 (VSS), JSODIMM2.99 (VSS), JSODIMM2.MP1, JSODIMM2.MP2
