File: Display_ports.kicad_sch (KiCad schematic)
At the start: 52 parts, among them J2 DP_A, J3 DP_B, J4 DP_C, J5 eDP 4-lane 40-pin ipex, Q1 2N7002, Q2 2N7002, Q3 2N7002, Q4 2N7002, Q5 2N7002, Q6 2N7002

Commit message: nooo they be stealin my stroopwafel
Connections:
- net at J5.36 (BL_PWR): now also J5.37 (BL_PWR), J5.38 (BL_PWR), J5.39 (BL_PWR)
Changed lines of the file:
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@@
+	)
+	(junction
+		(at 85.09 177.8)
+		(diameter 0)
+		(color 0 0 0 0)
 	)
 	(junction
@@
 	)
 	(junction
+		(at 85.09 175.26)
+		(diameter 0)
+		(color 0 0 0 0)
+	)
+	(junction
 		(at 356.87 199.39)
 		(diameter 0)
@@
 	(wire
 		(pts
+			(xy 85.09 175.26) (xy 85.09 177.8)
+		)
+		(stroke
+			(width 0)
+			(type default)
+		)
+	)
+	(wire
+		(pts
 			(xy 355.6 189.23) (xy 355.6 190.5)
 		)
@@
 	(wire
 		(pts
+			(xy 85.09 177.8) (xy 85.09 180.34)
+		)
+		(stroke
+			(width 0)
+			(type default)
+		)
+	)
+	(wire
+		(pts
 			(xy 231.14 36.83) (xy 232.41 36.83)
 		)
@@
 	(wire
 		(pts
+			(xy 85.09 172.72) (xy 87.63 172.72)
+		)
+		(stroke
+			(width 0)
+			(type default)
+		)
+	)
+	(wire
+		(pts
 			(xy 265.43 68.58) (xy 270.51 68.58)
 		)
@@
 	(wire
 		(pts
+			(xy 85.09 175.26) (xy 87.63 175.26)
+		)
+		(stroke
+			(width 0)
+			(type default)
+		)
+	)
+	(wire
+		(pts
 			(xy 190.5 53.34) (xy 190.5 55.88)
 		)
@@
 	(wire
 		(pts
+			(xy 85.09 172.72) (xy 85.09 175.26)
+		)
+		(stroke
+			(width 0)
+			(type default)
+		)
+	)
+	(wire
+		(pts
 			(xy 233.68 27.94) (xy 234.95 27.94)
 		)
@@
 	(wire
 		(pts
+			(xy 85.09 180.34) (xy 87.63 180.34)
+		)
+		(stroke
+			(width 0)
+			(type default)
+		)
+	)
+	(wire
+		(pts
 			(xy 330.2 55.88) (xy 355.6 55.88)
 		)
@@
 		)
 		(stroke
+			(width 0)
+			(type default)
+		)
+	)
+	(wire
+		(pts
+			(xy 85.09 177.8) (xy 87.63 177.8)
+		)
+		(stroke
