File: EC.kicad_sch (KiCad schematic)
At the start: 0 parts

Commit message: Added interconnect between CPU and PCH boards and added ATX board outline
Other:
- company: (none) -> WifiCable
- title: (none) -> Embedded Controller
Changed lines of the file:
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@@
 	(generator_version "9.0")
 	(paper "A4")
+	(title_block
+		(title "Embedded Controller")
+		(company "WifiCable")
+	)
 	(global_label "PECI_EC"
 		(shape input)
