File: PCIe_PCH.kicad_sch (KiCad schematic)
At the start: 18 parts, among them J6 Bus_M.2_Socket_M, J7 PCIe_x16_CPU

Commit message: Added more PCIe slots and mounting holes
Parts:
- added C100, C101, C102, C103, C104, C105, C106, C107, C108, C85, C86, C87, C88, C89, C90, C91, C92, C93, C94, C95, C96, C97, C98, C99: 0.22uF, Capacitor_SMD:C_0402_1005Metric, symbol Device:C_Small
- added J10: PCIe_x4_PCH_5, A-my-stuff:PCIe_x4_tht_open, symbol A-my-stuff:PCIe_x4_full
- added J11: PCIe_x4_PCH_4, A-my-stuff:PCIe_x4_tht_open, symbol A-my-stuff:PCIe_x4_full
- added J12: PCIe_x4_PCH_1, A-my-stuff:PCIe_x4_tht_open, symbol A-my-stuff:PCIe_x4_full
- J7: value PCIe_x16_CPU -> PCIe_x4_PCH_6
Connections:
- net GND: now also J10.A1 (~{PRSNT1}), J11.A1 (~{PRSNT1}), J12.A1 (~{PRSNT1})
- net temp_12V: now also J10.A2 (+12V), J10.A3 (+12V), J10.B1 (+12V), J10.B2 (+12V), J10.B3 (+12V), J11.A2 (+12V), J11.A3 (+12V), J11.B1 (+12V), J11.B2 (+12V), J11.B3 (+12V), J12.A2 (+12V), J12.A3 (+12V), J12.B1 (+12V), J12.B2 (+12V), J12.B3 (+12V)
- net temp_3.3V: now also J10.A10 (+3.3V), J10.A9 (+3.3V), J10.B8 (+3.3V), J11.A10 (+3.3V), J11.A9 (+3.3V), J11.B8 (+3.3V), J12.A10 (+3.3V), J12.A9 (+3.3V), J12.B8 (+3.3V)
- net PCH_x4_CLKREQ# renamed PCH_x4_6_CLKREQ#
- net PCH_x4_PCIe_C_Tx0+ renamed PCH_x4_6_PCIe_C_Tx0+
- net PCH_x4_PCIe_C_Tx0- renamed PCH_x4_6_PCIe_C_Tx0-
- net PCH_x4_PCIe_C_Tx1+ renamed PCH_x4_6_PCIe_C_Tx1+
- net PCH_x4_PCIe_C_Tx1- renamed PCH_x4_6_PCIe_C_Tx1-
- net PCH_x4_PCIe_C_Tx2+ renamed PCH_x4_6_PCIe_C_Tx2+
- net PCH_x4_PCIe_C_Tx2- renamed PCH_x4_6_PCIe_C_Tx2-
- net PCH_x4_PCIe_C_Tx3+ renamed PCH_x4_6_PCIe_C_Tx3+
- net PCH_x4_PCIe_C_Tx3- renamed PCH_x4_6_PCIe_C_Tx3-
- net PCH_x4_PCIe_Rx0+ renamed PCH_x4_6_PCIe_Rx0+
- net PCH_x4_PCIe_Rx0- renamed PCH_x4_6_PCIe_Rx0-
- net PCH_x4_PCIe_Rx1+ renamed PCH_x4_6_PCIe_Rx1+
- net PCH_x4_PCIe_Rx1- renamed PCH_x4_6_PCIe_Rx1-
- net PCH_x4_PCIe_Rx2+ renamed PCH_x4_6_PCIe_Rx2+
- net PCH_x4_PCIe_Rx2- renamed PCH_x4_6_PCIe_Rx2-
- net PCH_x4_PCIe_Rx3+ renamed PCH_x4_6_PCIe_Rx3+
- net PCH_x4_PCIe_Rx3- renamed PCH_x4_6_PCIe_Rx3-
- net PCH_x4_PCIe_Tx0+ renamed PCH_x4_6_PCIe_Tx0+
- net PCH_x4_PCIe_Tx0- renamed PCH_x4_6_PCIe_Tx0-
- net PCH_x4_PCIe_Tx1+ renamed PCH_x4_6_PCIe_Tx1+
- net PCH_x4_PCIe_Tx1- renamed PCH_x4_6_PCIe_Tx1-
- net PCH_x4_PCIe_Tx2+ renamed PCH_x4_6_PCIe_Tx2+
- net PCH_x4_PCIe_Tx2- renamed PCH_x4_6_PCIe_Tx2-
- net PCH_x4_PCIe_Tx3+ renamed PCH_x4_6_PCIe_Tx3+
- net PCH_x4_PCIe_Tx3- renamed PCH_x4_6_PCIe_Tx3-
- net PCH_x4_Refclk+ renamed PCH_x4_6_Refclk+
- net PCH_x4_Refclk- renamed PCH_x4_6_Refclk-
- net SSD0_PCIe/SATA_C_Tx0+ renamed SSD0_SATA/PCIe_C_Tx0+
- net SSD0_PCIe/SATA_C_Tx0- renamed SSD0_SATA/PCIe_C_Tx0-
- net SSD0_PCIe/SATA_Rx0+ renamed SSD0_SATA/PCIe_Rx0+
- net SSD0_PCIe/SATA_Rx0- renamed SSD0_SATA/PCIe_Rx0-
- net SSD0_PCIe/SATA_Tx0+ renamed SSD0_SATA/PCIe_Tx0+
- net SSD0_PCIe/SATA_Tx0- renamed SSD0_SATA/PCIe_Tx0-
- new net: J11.A12 (GND), J11.A15 (GND), J11.A18 (GND), J11.A20 (GND), J11.A23 (GND), J11.A24 (GND), J11.A27 (GND), J11.A28 (GND), J11.A31 (GND), J11.A4 (GND)
- new net: J11.B13 (GND), J11.B16 (GND), J11.B18 (GND), J11.B21 (GND), J11.B22 (GND), J11.B25 (GND), J11.B26 (GND), J11.B29 (GND), J11.B32 (GND), J11.B4 (GND), J11.B7 (GND)
- new net: J12.A12 (GND), J12.A15 (GND), J12.A18 (GND), J12.A20 (GND), J12.A23 (GND), J12.A24 (GND), J12.A27 (GND), J12.A28 (GND), J12.A31 (GND), J12.A4 (GND)
- new net: J12.B13 (GND), J12.B16 (GND), J12.B18 (GND), J12.B21 (GND), J12.B22 (GND), J12.B25 (GND), J12.B26 (GND), J12.B29 (GND), J12.B32 (GND), J12.B4 (GND), J12.B7 (GND)
- new net: J10.A12 (GND), J10.A15 (GND), J10.A18 (GND), J10.A20 (GND), J10.A23 (GND), J10.A24 (GND), J10.A27 (GND), J10.A28 (GND), J10.A31 (GND), J10.A4 (GND)
- new net: J10.B13 (GND), J10.B16 (GND), J10.B18 (GND), J10.B21 (GND), J10.B22 (GND), J10.B25 (GND), J10.B26 (GND), J10.B29 (GND), J10.B32 (GND), J10.B4 (GND), J10.B7 (GND)
- new net PCH_x4_1_CLKREQ#: J12.B17 (~{PRSNT2}), J12.B31 (~{PRSNT2})
- new net PCH_x4_1_PCIe_C_Tx0+: C101.2, J12.B14 (PETp0)
- new net PCH_x4_1_PCIe_C_Tx0-: C102.2, J12.B15 (PETn0)
- new net PCH_x4_1_PCIe_C_Tx1+: C103.2, J12.B19 (PETp1)
- new net PCH_x4_1_PCIe_C_Tx1-: C104.2, J12.B20 (PETn1)
- new net PCH_x4_1_PCIe_C_Tx2+: C105.2, J12.B23 (PETp2)
- new net PCH_x4_1_PCIe_C_Tx2-: C106.2, J12.B24 (PETn2)
- new net PCH_x4_1_PCIe_C_Tx3+: C107.2, J12.B27 (PETp3)
- new net PCH_x4_1_PCIe_C_Tx3-: C108.2, J12.B28 (PETn3)
- new net PCH_x4_1_PCIe_Rx0+: J12.A16 (PERp0)
- new net PCH_x4_1_PCIe_Rx0-: J12.A17 (PERn0)
- new net PCH_x4_1_PCIe_Rx1+: J12.A21 (PERp1)
- new net PCH_x4_1_PCIe_Rx1-: J12.A22 (PERn1)
- new net PCH_x4_1_PCIe_Rx2+: J12.A25 (PERp2)
- new net PCH_x4_1_PCIe_Rx2-: J12.A26 (PERn2)
- new net PCH_x4_1_PCIe_Rx3+: J12.A29 (PERp3)
- new net PCH_x4_1_PCIe_Rx3-: J12.A30 (PERn3)
- new net PCH_x4_1_PCIe_Tx0+: C101.1
- new net PCH_x4_1_PCIe_Tx0-: C102.1
- new net PCH_x4_1_PCIe_Tx1+: C103.1
- new net PCH_x4_1_PCIe_Tx1-: C104.1
- new net PCH_x4_1_PCIe_Tx2+: C105.1
- new net PCH_x4_1_PCIe_Tx2-: C106.1
- new net PCH_x4_1_PCIe_Tx3+: C107.1
- new net PCH_x4_1_PCIe_Tx3-: C108.1
- new net PCH_x4_1_Refclk+: J12.A13 (REFCLK+)
- new net PCH_x4_1_Refclk-: J12.A14 (REFCLK-)
- new net PCH_x4_4_CLKREQ#: J11.B17 (~{PRSNT2}), J11.B31 (~{PRSNT2})
- new net PCH_x4_4_PCIe_C_Tx0+: C93.2, J11.B14 (PETp0)
- new net PCH_x4_4_PCIe_C_Tx0-: C94.2, J11.B15 (PETn0)
- new net PCH_x4_4_PCIe_C_Tx1+: C95.2, J11.B19 (PETp1)
- new net PCH_x4_4_PCIe_C_Tx1-: C96.2, J11.B20 (PETn1)
- new net PCH_x4_4_PCIe_C_Tx2+: C97.2, J11.B23 (PETp2)
- new net PCH_x4_4_PCIe_C_Tx2-: C98.2, J11.B24 (PETn2)
- new net PCH_x4_4_PCIe_C_Tx3+: C99.2, J11.B27 (PETp3)
- new net PCH_x4_4_PCIe_C_Tx3-: C100.2, J11.B28 (PETn3)
- new net PCH_x4_4_PCIe_Rx0+: J11.A16 (PERp0)
- new net PCH_x4_4_PCIe_Rx0-: J11.A17 (PERn0)
- new net PCH_x4_4_PCIe_Rx1+: J11.A21 (PERp1)
- new net PCH_x4_4_PCIe_Rx1-: J11.A22 (PERn1)
- new net PCH_x4_4_PCIe_Rx2+: J11.A25 (PERp2)
- new net PCH_x4_4_PCIe_Rx2-: J11.A26 (PERn2)
- new net PCH_x4_4_PCIe_Rx3+: J11.A29 (PERp3)
- new net PCH_x4_4_PCIe_Rx3-: J11.A30 (PERn3)
- new net PCH_x4_4_PCIe_Tx0+: C93.1
- new net PCH_x4_4_PCIe_Tx0-: C94.1
- new net PCH_x4_4_PCIe_Tx1+: C95.1
- new net PCH_x4_4_PCIe_Tx1-: C96.1
- new net PCH_x4_4_PCIe_Tx2+: C97.1
- new net PCH_x4_4_PCIe_Tx2-: C98.1
- new net PCH_x4_4_PCIe_Tx3+: C99.1
- new net PCH_x4_4_PCIe_Tx3-: C100.1
- new net PCH_x4_4_Refclk+: J11.A13 (REFCLK+)
- new net PCH_x4_4_Refclk-: J11.A14 (REFCLK-)
- new net PCH_x4_5_CLKREQ#: J10.B17 (~{PRSNT2}), J10.B31 (~{PRSNT2})
- new net PCH_x4_5_PCIe_C_Tx0+: C85.2, J10.B14 (PETp0)
- new net PCH_x4_5_PCIe_C_Tx0-: C86.2, J10.B15 (PETn0)
- new net PCH_x4_5_PCIe_C_Tx1+: C87.2, J10.B19 (PETp1)
- new net PCH_x4_5_PCIe_C_Tx1-: C88.2, J10.B20 (PETn1)
- new net PCH_x4_5_PCIe_C_Tx2+: C89.2, J10.B23 (PETp2)
- new net PCH_x4_5_PCIe_C_Tx2-: C90.2, J10.B24 (PETn2)
- new net PCH_x4_5_PCIe_C_Tx3+: C91.2, J10.B27 (PETp3)
- new net PCH_x4_5_PCIe_C_Tx3-: C92.2, J10.B28 (PETn3)
- new net PCH_x4_5_PCIe_Rx0+: J10.A16 (PERp0)
- new net PCH_x4_5_PCIe_Rx0-: J10.A17 (PERn0)
- new net PCH_x4_5_PCIe_Rx1+: J10.A21 (PERp1)
- new net PCH_x4_5_PCIe_Rx1-: J10.A22 (PERn1)
- new net PCH_x4_5_PCIe_Rx2+: J10.A25 (PERp2)
- new net PCH_x4_5_PCIe_Rx2-: J10.A26 (PERn2)
- new net PCH_x4_5_PCIe_Rx3+: J10.A29 (PERp3)
- new net PCH_x4_5_PCIe_Rx3-: J10.A30 (PERn3)
- new net PCH_x4_5_PCIe_Tx0+: C85.1
- new net PCH_x4_5_PCIe_Tx0-: C86.1
- new net PCH_x4_5_PCIe_Tx1+: C87.1
- new net PCH_x4_5_PCIe_Tx1-: C88.1
- new net PCH_x4_5_PCIe_Tx2+: C89.1
- new net PCH_x4_5_PCIe_Tx2-: C90.1
- new net PCH_x4_5_PCIe_Tx3+: C91.1
- new net PCH_x4_5_PCIe_Tx3-: C92.1
- new net PCH_x4_5_Refclk+: J10.A13 (REFCLK+)
- new net PCH_x4_5_Refclk-: J10.A14 (REFCLK-)
- no-connect marks 1 -> 4
Other:
- moved on the sheet: C69, C70, C71, C72, C73, C74, C75, C76, C77, C78, C79, C80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
